File: easyL1105_KiCad_source/MSPM0L1105_dev_board.kicad_pcb (KiCad board)
At the start: 2 copper layers, 61 x 38.1 mm, 45 parts, among them J1 IO_A, J2 IO_B, J3 UART-SELECT, J4 USB_C_Receptacle_USB4085, J5 SWD, J6 LDO_JUMPER, J7 GND_JUMPER, SW1 RESET, SW2 BSL_BOOT, SW3 USER_PA16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

Commit message: Rev 2.0
Parts:
- removed R16, R18: 10k, Resistor_SMD:R_0805_2012Metric_Pad1.20x1.40mm_HandSolder
- removed R6: DNF, Resistor_SMD:R_0805_2012Metric_Pad1.20x1.40mm_HandSolder
- added D5: BAS16, User_Global_Library:SOT-23-NEW, F.Cu at (115.2, 55.4)
- added D6: BAS16, User_Global_Library:SOT-23-NEW, B.Cu at (75.6, 64.4)
- added Q3: BC857, User_Global_Library:SOT-23-NEW, F.Cu at (115.3, 59.1)
- added R17: 100k, Resistor_SMD:R_0805_2012Metric_Pad1.20x1.40mm_HandSolder, F.Cu at (88.4, 60.3)
- added R24: 47k, Resistor_SMD:R_0805_2012Metric_Pad1.20x1.40mm_HandSolder, F.Cu at (109.3, 77.0)
- added R25: 10k, Resistor_SMD:R_0805_2012Metric_Pad1.20x1.40mm_HandSolder, F.Cu at (112.3, 59.2)
- added R26: 10k, Resistor_SMD:R_0805_2012Metric_Pad1.20x1.40mm_HandSolder, F.Cu at (112.3, 55.4)
- added R27: 10k, Resistor_SMD:R_0805_2012Metric_Pad1.20x1.40mm_HandSolder, B.Cu at (76.6, 71.2)
- D1: value PA27 -> GREEN
- D2: value PA26 -> BLUE
- D4: value PWR -> RED
- R10: value 470R -> 220R
- R11: value 470R -> 820R
- R19: value 470R -> 1k
- R7: value DNF -> 100k
- moved R7 4.99 mm to (118.2, 59.2), turned to -90 degrees
- moved R4 3.02 mm to (114.9, 52.4)
- moved J5 2.54 mm to (116.8, 73.7)
Connections:
- J2 pad 2: /PA9 -> /BSL_INVOKE
- J3 pad 1: /RXD -> Net-(D6-A)
- J3 pad 5: /RXD -> Net-(D6-A)
- R3 pad 2: Net-(U1-RXD/BSL_INVOKE/PA18/A7) -> /PA9
- R7 pad 1: 0V -> /BSL_INVOKE
- R7 pad 2: Net-(U1-RXD/BSL_INVOKE/PA18/A7) -> 0V
- SW2 pad 1: Net-(U1-RXD/BSL_INVOKE/PA18/A7) -> /BSL_INVOKE
- U1 pad 21: Net-(U1-RXD/BSL_INVOKE/PA18/A7) -> /BSL_INVOKE
- U2 pad 4: unconnected-(U2-~{DTR}-Pad4) -> /*DTR
Routing:
- net /*DTR: track 0.00 -> 74.6 mm
- net Net-(U1-RXD/BSL_INVOKE/PA18/A7): track 36.4 -> 0.00 mm, vias 4 -> 0
- net /BSL_INVOKE: track 0.00 -> 36.0 mm, vias 0 -> 2
- net +3.3V: track 214.4 -> 242.9 mm, vias 1 -> 2
- net Net-(D6-A): track 0.00 -> 17.2 mm
- net /BSL_RX: track 26.7 -> 16.4 mm
- net /*RST: track 38.6 -> 48.3 mm
- net /UART0_TXD: track 4.69 -> 13.8 mm
- net /RXD: track 19.1 -> 11.3 mm
- net Net-(D5-K): track 0.00 -> 7.49 mm
- net /SWDIO: track 54.6 -> 58.6 mm
- net Net-(Q3-B): track 0.00 -> 3.84 mm
- net /SWCLK: track 33.9 -> 37.2 mm
- net /PA9: track 21.0 -> 23.9 mm, vias 0 -> 2
- net /UART0_RXD: track 6.44 -> 4.81 mm
Other:
- board size 61 x 38.1 mm -> 64.9 x 38.1 mm
- board text added: "0V"
- board text added: "CLK"
- board text added: "DIO"
- board text added: "REV 2.0"
- board text added: "Rev 2.0"
- board text removed: "PA9"
- board text removed: "REV 1.0"
