File: easyL1105_KiCad_source/MSPM0L1105_dev_board.kicad_sch (KiCad schematic)
At the start: 51 parts, among them J1 IO_A, J2 IO_B, J3 UART-SELECT, J4 USB_C_Receptacle_USB4085, J5 SWD, J6 LDO_JUMPER, J7 GND_JUMPER, SW1 RESET, SW2 BSL_BOOT, SW3 USER_PA16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

Commit message: Add files via upload
Parts:
- D1: value PA27 -> GREEN
- D2: value PA26 -> BLUE
- R18: value 10k -> DNF
- R7: value DNF -> 100k
Other:
- moved on the sheet: J5, R4, R5

Commit message: Rev 2.0
Parts:
- removed R16: 10k, Resistor_SMD:R_0805_2012Metric_Pad1.20x1.40mm_HandSolder, symbol Device:R
- removed R18, R6: DNF, Resistor_SMD:R_0805_2012Metric_Pad1.20x1.40mm_HandSolder, symbol Device:R
- added D5, D6: BAS16, User_Global_Library:SOT-23-NEW, symbol User_Global_Symbol_Library:BAS16
- added Q3: BC857, User_Global_Library:SOT-23-NEW, symbol User_Global_Symbol_Library:BC857
- added R17: 100k, Resistor_SMD:R_0805_2012Metric_Pad1.20x1.40mm_HandSolder, symbol Device:R
- added R24: 47k, Resistor_SMD:R_0805_2012Metric_Pad1.20x1.40mm_HandSolder, symbol Device:R
- added R25, R26, R27: 10k, Resistor_SMD:R_0805_2012Metric_Pad1.20x1.40mm_HandSolder, symbol Device:R
- added TEXT3, TEXT8: arrow, symbol User_Global_Symbol_Library:arrow
- D4: value PWR -> RED
- R10: value 470R -> 220R
- R11: value 470R -> 820R
- R19: value 470R -> 1k
- U1: symbol User_Global_Symbol_Library:MSPM0L1105TDGS28R -> User_Global_Symbol_Library:MSPM0L1105TDGS28R_NEW_ARRANGEMENT
Connections:
- net *RST: now also R24.2
- net +3.3V: now also D5.1 (A), R17.1, R24.1, R27.1
- net 0V: now also R7.2; no longer R7.1
- net PA9: now also R3.2; no longer J2.2 (Pin_2)
- net RXD: now also D6.3 (K); no longer J3.1 (Pin_1), J3.5 (Pin_5)
- net UART0_TXD: now also R17.2
- net BSL_INVOKE: now reaches SW2.1, U1.21 (BSL_INVOKE/PA18)
- net BSL_INVOKE: now also J2.2 (Pin_2), R7.1, Q3.3 (C); no longer R3.2, R7.2
- net *DTR: now reaches U2.4 (~{DTR})
- net *DTR: now also R26.1
- new net: D5.3 (K), Q3.2 (E), R25.1
- new net: D6.1 (A), J3.1 (Pin_1), J3.5 (Pin_5), R27.2
- new net: Q3.1 (B), R25.2, R26.2
- no-connect marks 6 -> 5
Other:
- note added: "2"
- note added: "AUTO-BOOTLOADER"
- note added: "AUTO-RESET"
- note added: "EasyL1105 MSPM0L1105 Dev Board"
- note removed: "1"
- note removed: "MSPM0L1105 Dev Board"
- moved on the sheet: C1, C2, C3, C4, C5, C6, C7, C8, C9, D1, D2, D3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
